File: ridhaulakbar75.sch (KiCad schematic (older format))
At the start: 202 parts, among them J1 AVR-ISP-6, J2 Conn_01x04, U1 TEENSY2.0

Commit message: update
Parts:
- removed R1, R2: 5.1K, Resistor_SMD:R_0805_2012Metric_Pad1.15x1.40mm_HandSolder, symbol Device:R_Small
- added C18, C9: 0.1uF, Capacitor_SMD:C_0603_1608Metric_Pad1.05x0.95mm_HandSolder, symbol Device:C_Small
- added LED18, LED9: WS2812B, WS2812B:WS2812B, symbol ws2812b:WS2812B
- renumbered C2 to C10, C4 to C11, C6 to C12, C8 to C13, C10 to C14, C12 to C15, C14 to C16, C16 to C17, C3 to C2, C5 to C3, C7 to C4, C9 to C5, C11 to C6, C13 to C7, C15 to C8, D16 to D11, D11 to D12, D12 to D13, D13 to D14, D14 to D15, D15 to D16, D27 to D22, D22 to D23, D23 to D24, D24 to D25, D25 to D26, D26 to D27, D55 to D54, D56 to D55, D57 to D56, D58 to D57, D59 to D58, D54 to D59, D61 to D60, D62 to D61, D63 to D62, D64 to D63, D65 to D64, D66 to D65, D67 to D66, D68 to D67, D69 to D68, D71 to D69, D72 to D70, D73 to D71, D74 to D72, D75 to D73, D70 to D74, D76 to D75, D77 to D76, D78 to D77, D79 to D78, D80 to D79, D81 to D80, D82 to D81, D83 to D82, J2 to J1, J1 to J2, LED9 to LED10, LED10 to LED11, LED11 to LED12, LED12 to LED13, LED13 to LED14, LED14 to LED15, LED15 to LED16, LED16 to LED17, MX16 to MX11, MX11 to MX12, MX12 to MX13, MX13 to MX14, MX14 to MX15, MX15 to MX16, MX27 to MX22, MX22 to MX23, MX23 to MX24, MX24 to MX25, MX25 to MX26, MX26 to MX27, MX55 to MX54, MX56 to MX55, MX57 to MX56, MX58 to MX57, MX59 to MX58, MX54 to MX59, MX61 to MX60, MX62 to MX61, MX63 to MX62, MX64 to MX63, MX65 to MX64, MX66 to MX65, MX67 to MX66, MX68 to MX67, MX69 to MX68, MX71 to MX69, MX72 to MX70, MX73 to MX71, MX74 to MX72, MX75 to MX73, MX70 to MX74, MX76 to MX75, MX77 to MX76, MX78 to MX77, MX79 to MX78, MX80 to MX79, MX81 to MX80, MX82 to MX81, MX83 to MX82
Connections:
- net labels added: D+, D-, VBUS
- wire segments 498 -> 506

Commit message: big update
Parts:
- removed C1, C10, C11, C12, C13, C14, C15, C16, C17, C18, C2, C3, C4, C5, C6, C7, C8, C9: 0.1uF, Capacitor_SMD:C_0603_1608Metric_Pad1.05x0.95mm_HandSolder, symbol Device:C_Small
- removed D71: 1N4148W, master-Keebio-Parts:D_SOD-123-v2, symbol Diode:1N4148W
- removed J2: AVR-ISP-6, random-keyboard-parts:Reset_Pretty-Mask, symbol Connector:AVR-ISP-6
- removed LED1, LED10, LED11, LED12, LED13, LED14, LED15, LED16, LED17, LED18, LED2, LED3, LED4, LED5, LED6, LED7, LED8, LED9: WS2812B, WS2812B:WS2812B, symbol ws2812b:WS2812B
- removed MX71: Prnt Scr, MX_Only:MXOnly-1U-NoLED, symbol MX_Alps_Hybrid:MX-NoLED
- removed U1: TEENSY2.0, master-Keebio-Parts:Teensy_2.0, symbol keyboard_parts:TEENSY2.0
- added D82: BLUE, LED_SMD:LED_0603_1608Metric, symbol Device:LED
- added D83: 1N5819, Diode_SMD:D_SOD-323F, symbol Device:D_Schottky_Small
- added D84: RED, LED_SMD:LED_0603_1608Metric, symbol Device:LED
- added F1: 500mA, Fuse:Fuse_1206_3216Metric, symbol Device:Polyfuse_Small
- added J2: Ex_Bat, Connector_PinHeader_2.54mm:PinHeader_1x02_P2.54mm_Vertical, symbol Connector_Generic:Conn_01x02
- added J3: Ex_USB, nrfmicro:connector_usb, symbol Connector_Generic:Conn_01x04
- added Q1, Q2: AO3407, Package_TO_SOT_SMD:SOT-23, symbol Device:Q_PMOS_GSD
- added R1, R2: 5.1k, Resistor_SMD:R_0603_1608Metric, symbol Device:R_Small
- added R3: 820K, Resistor_SMD:R_0603_1608Metric, symbol Device:R_Small
- added R4, R8: 1K, Resistor_SMD:R_0603_1608Metric, symbol Device:R_Small
- added R5, R6: 2M, Resistor_SMD:R_0603_1608Metric, symbol Device:R_Small
- added R7: 100k, Resistor_SMD:R_0603_1608Metric, symbol Device:R_Small
- added R9: 2K, Resistor_SMD:R_0603_1608Metric, symbol Device:R_Small
- added SW1: Rotary_Encoder_Switch, master-Keebio-Parts:RotaryEncoder_EC11-no-legs, symbol Device:Rotary_Encoder_Switch
- added U1: USBLC6-2SC6, Package_TO_SOT_SMD:SOT-23-6, symbol Power_Protection:USBLC6-2SC6
- added U2: E73-2G4M08S1C-52840, nrfmicro:E73-2G4M08S1C-52840, symbol nrfmicro:E73-2G4M08S1C-52840
- added U3: XC6220B331MR, Package_TO_SOT_SMD:SOT-23-5, symbol Regulator_Linear:XC6220B331MR
- added U4: TP4054, Package_TO_SOT_SMD:SOT-23-5, symbol Battery_Management:MCP73831-3-OT
- added Y1: 32.768kHz, Crystal:Crystal_SMD_MicroCrystal_CM9V-T1A-2Pin_1.6x1.0mm, symbol Device:Crystal_Small
- J1: value Conn_01x04 -> SWD; footprint Connector_PinHeader_2.54mm:PinHeader_1x04_P2.54mm_Vertical -> nrfmicro:connector_swd
- MX1, MX18: footprint MX_Only:MXOnly-1U-NoLED -> MX_Only:MXOnly-1U-Hotswap
- MX10: renamed from MX49; footprint MX_Only:MXOnly-1U-NoLED -> MX_Only:MXOnly-1U-Hotswap
- MX11: renamed from MX54; footprint MX_Only:MXOnly-1U-NoLED -> MX_Only:MXOnly-1U-Hotswap
- MX12: renamed from MX60; footprint MX_Only:MXOnly-1U-NoLED -> MX_Only:MXOnly-1U-Hotswap
- MX13: renamed from MX66; footprint MX_Only:MXOnly-1U-NoLED -> MX_Only:MXOnly-1U-Hotswap
- MX14: renamed from MX77; footprint MX_Only:MXOnly-1U-NoLED -> MX_Only:MXOnly-1U-Hotswap
- MX15: renamed from MX2; footprint MX_Only:MXOnly-1U-NoLED -> MX_Only:MXOnly-1U-Hotswap
- MX16: renamed from MX8; footprint MX_Only:MXOnly-1U-NoLED -> MX_Only:MXOnly-1U-Hotswap
- MX17: renamed from MX13; footprint MX_Only:MXOnly-1U-NoLED -> MX_Only:MXOnly-1U-Hotswap
- MX19: renamed from MX24; footprint MX_Only:MXOnly-1U-NoLED -> MX_Only:MXOnly-1U-Hotswap
- MX2: renamed from MX7; footprint MX_Only:MXOnly-1U-NoLED -> MX_Only:MXOnly-1U-Hotswap
- MX20: renamed from MX29; footprint MX_Only:MXOnly-1U-NoLED -> MX_Only:MXOnly-1U-Hotswap
- MX21: renamed from MX34; footprint MX_Only:MXOnly-1U-NoLED -> MX_Only:MXOnly-1U-Hotswap
- MX22: renamed from MX40; footprint MX_Only:MXOnly-1U-NoLED -> MX_Only:MXOnly-1U-Hotswap
- MX23: renamed from MX45; footprint MX_Only:MXOnly-1U-NoLED -> MX_Only:MXOnly-1U-Hotswap
- MX24: renamed from MX50; footprint MX_Only:MXOnly-1U-NoLED -> MX_Only:MXOnly-1U-Hotswap
- MX25: renamed from MX55; footprint MX_Only:MXOnly-1U-NoLED -> MX_Only:MXOnly-1U-Hotswap
- MX26: renamed from MX61; footprint MX_Only:MXOnly-1U-NoLED -> MX_Only:MXOnly-1U-Hotswap
- MX27: renamed from MX67; footprint MX_Only:MXOnly-1U-NoLED -> MX_Only:MXOnly-1U-Hotswap
- MX28: renamed from MX72; footprint MX_Only:MXOnly-2U-NoLED -> MX_Only:MXOnly-2U-Hotswap
- MX29: renamed from MX78; footprint MX_Only:MXOnly-1U-NoLED -> MX_Only:MXOnly-1U-Hotswap
- MX3: renamed from MX12; footprint MX_Only:MXOnly-1U-NoLED -> MX_Only:MXOnly-1U-Hotswap
- MX30: renamed from MX3; footprint MX_Only:MXOnly-1.5U-NoLED -> MX_Only:MXOnly-1.5U-Hotswap
- MX31: renamed from MX9; footprint MX_Only:MXOnly-1U-NoLED -> MX_Only:MXOnly-1U-Hotswap
- MX32: renamed from MX14; footprint MX_Only:MXOnly-1U-NoLED -> MX_Only:MXOnly-1U-Hotswap
- MX33: renamed from MX19; footprint MX_Only:MXOnly-1U-NoLED -> MX_Only:MXOnly-1U-Hotswap
- MX34: renamed from MX25; footprint MX_Only:MXOnly-1U-NoLED -> MX_Only:MXOnly-1U-Hotswap
- MX35: renamed from MX30; footprint MX_Only:MXOnly-1U-NoLED -> MX_Only:MXOnly-1U-Hotswap
- MX36: renamed from MX35; footprint MX_Only:MXOnly-1U-NoLED -> MX_Only:MXOnly-1U-Hotswap
- MX37: renamed from MX41; footprint MX_Only:MXOnly-1U-NoLED -> MX_Only:MXOnly-1U-Hotswap
- MX38: renamed from MX46; footprint MX_Only:MXOnly-1U-NoLED -> MX_Only:MXOnly-1U-Hotswap
- MX39: renamed from MX51; footprint MX_Only:MXOnly-1U-NoLED -> MX_Only:MXOnly-1U-Hotswap
- MX4: renamed from MX17; footprint MX_Only:MXOnly-1U-NoLED -> MX_Only:MXOnly-1U-Hotswap
- MX40: renamed from MX56; footprint MX_Only:MXOnly-1U-NoLED -> MX_Only:MXOnly-1U-Hotswap
- MX41: renamed from MX62; footprint MX_Only:MXOnly-1U-NoLED -> MX_Only:MXOnly-1U-Hotswap
- MX42: renamed from MX68; footprint MX_Only:MXOnly-1U-NoLED -> MX_Only:MXOnly-1U-Hotswap
- MX43: renamed from MX73; footprint MX_Only:MXOnly-1.5U-NoLED -> MX_Only:MXOnly-1.5U-Hotswap
- MX44: renamed from MX79; footprint MX_Only:MXOnly-1U-NoLED -> MX_Only:MXOnly-1U-Hotswap
- MX45: renamed from MX4; footprint MX_Only:MXOnly-1.75U-NoLED -> MX_Only:MXOnly-1.75U-Hotswap
- MX46: renamed from MX10; footprint MX_Only:MXOnly-1U-NoLED -> MX_Only:MXOnly-1U-Hotswap
- MX47: renamed from MX15; footprint MX_Only:MXOnly-1U-NoLED -> MX_Only:MXOnly-1U-Hotswap
- MX48: renamed from MX20; footprint MX_Only:MXOnly-1U-NoLED -> MX_Only:MXOnly-1U-Hotswap
- MX49: renamed from MX26; footprint MX_Only:MXOnly-1U-NoLED -> MX_Only:MXOnly-1U-Hotswap
- MX5: renamed from MX23; footprint MX_Only:MXOnly-1U-NoLED -> MX_Only:MXOnly-1U-Hotswap
- MX50: renamed from MX31; footprint MX_Only:MXOnly-1U-NoLED -> MX_Only:MXOnly-1U-Hotswap
- MX51: renamed from MX36; footprint MX_Only:MXOnly-1U-NoLED -> MX_Only:MXOnly-1U-Hotswap
- MX52: renamed from MX42; footprint MX_Only:MXOnly-1U-NoLED -> MX_Only:MXOnly-1U-Hotswap
- MX53: renamed from MX47; footprint MX_Only:MXOnly-1U-NoLED -> MX_Only:MXOnly-1U-Hotswap
- MX54: renamed from MX52; footprint MX_Only:MXOnly-1U-NoLED -> MX_Only:MXOnly-1U-Hotswap
- MX55: renamed from MX57; footprint MX_Only:MXOnly-1U-NoLED -> MX_Only:MXOnly-1U-Hotswap
- MX56: renamed from MX63; footprint MX_Only:MXOnly-1U-NoLED -> MX_Only:MXOnly-1U-Hotswap
- MX57: renamed from MX74; footprint MX_Only:MXOnly-2.25U-NoLED -> MX_Only:MXOnly-2.25U-Hotswap
- MX58: renamed from MX80; footprint MX_Only:MXOnly-1U-NoLED -> MX_Only:MXOnly-1U-Hotswap
- MX59: renamed from MX5; footprint MX_Only:MXOnly-2.25U-NoLED -> MX_Only:MXOnly-2.25U-Hotswap
- MX6: renamed from MX28; footprint MX_Only:MXOnly-1U-NoLED -> MX_Only:MXOnly-1U-Hotswap
- MX60: renamed from MX16; footprint MX_Only:MXOnly-1U-NoLED -> MX_Only:MXOnly-1U-Hotswap
- MX61: renamed from MX21; footprint MX_Only:MXOnly-1U-NoLED -> MX_Only:MXOnly-1U-Hotswap
- MX62: renamed from MX27; footprint MX_Only:MXOnly-1U-NoLED -> MX_Only:MXOnly-1U-Hotswap
- MX63: renamed from MX32; footprint MX_Only:MXOnly-1U-NoLED -> MX_Only:MXOnly-1U-Hotswap
- MX64: renamed from MX37; footprint MX_Only:MXOnly-1U-NoLED -> MX_Only:MXOnly-1U-Hotswap
- MX65: renamed from MX43; footprint MX_Only:MXOnly-1U-NoLED -> MX_Only:MXOnly-1U-Hotswap
- MX66: renamed from MX48; footprint MX_Only:MXOnly-1U-NoLED -> MX_Only:MXOnly-1U-Hotswap
- MX67: renamed from MX53; footprint MX_Only:MXOnly-1U-NoLED -> MX_Only:MXOnly-1U-Hotswap
- MX68: renamed from MX58; footprint MX_Only:MXOnly-1U-NoLED -> MX_Only:MXOnly-1U-Hotswap
- MX69: renamed from MX64; footprint MX_Only:MXOnly-1U-NoLED -> MX_Only:MXOnly-1U-Hotswap
- MX7: renamed from MX33; footprint MX_Only:MXOnly-1U-NoLED -> MX_Only:MXOnly-1U-Hotswap
- MX70: renamed from MX69; footprint MX_Only:MXOnly-1.75U-NoLED -> MX_Only:MXOnly-1.75U-Hotswap
- MX71: renamed from MX75; footprint MX_Only:MXOnly-1U-NoLED -> MX_Only:MXOnly-1U-Hotswap
- MX72: renamed from MX81; footprint MX_Only:MXOnly-1U-NoLED -> MX_Only:MXOnly-1U-Hotswap
- MX73: renamed from MX6; footprint MX_Only:MXOnly-1.5U-NoLED -> MX_Only:MXOnly-1.25U-Hotswap
- MX74: renamed from MX11; footprint MX_Only:MXOnly-1U-NoLED -> MX_Only:MXOnly-1.25U-Hotswap
- MX75: renamed from MX22; footprint MX_Only:MXOnly-1.5U-NoLED -> MX_Only:MXOnly-1.25U-Hotswap
- MX76: renamed from MX38; footprint MX_Only:MXOnly-7U-NoLED -> MX_Only:MXOnly-6.25U-Hotswap-ReversedStabilizers
- MX77: renamed from MX59; footprint MX_Only:MXOnly-1U-NoLED -> MX_Only:MXOnly-1.25U-Hotswap
- MX78: renamed from MX65; footprint MX_Only:MXOnly-1U-NoLED -> MX_Only:MXOnly-1.25U-Hotswap
- MX79: renamed from MX70; footprint MX_Only:MXOnly-1U-NoLED -> MX_Only:MXOnly-1U-Hotswap
- MX8: renamed from MX39; footprint MX_Only:MXOnly-1U-NoLED -> MX_Only:MXOnly-1U-Hotswap
- MX80: renamed from MX76; footprint MX_Only:MXOnly-1U-NoLED -> MX_Only:MXOnly-1U-Hotswap
- MX81: renamed from MX82; footprint MX_Only:MXOnly-1U-NoLED -> MX_Only:MXOnly-1U-Hotswap
- MX9: renamed from MX44; footprint MX_Only:MXOnly-1U-NoLED -> MX_Only:MXOnly-1U-Hotswap
- USB1: footprint master-Keebio-Parts:HRO-TYPE-C-31-M-12-Assembly -> Type-C:HRO-TYPE-C-31-M-12-HandSoldering
- renumbered D49 to D10, D54 to D11, D60 to D12, D66 to D13, D77 to D14, D2 to D15, D8 to D16, D13 to D17, D24 to D19, D7 to D2, D29 to D20, D34 to D21, D40 to D22, D45 to D23, D50 to D24, D55 to D25, D61 to D26, D67 to D27, D72 to D28, D78 to D29, D12 to D3, D3 to D30, D9 to D31, D14 to D32, D19 to D33, D25 to D34, D30 to D35, D35 to D36, D41 to D37, D46 to D38, D51 to D39, D17 to D4, D56 to D40, D62 to D41, D68 to D42, D73 to D43, D79 to D44, D4 to D45, D10 to D46, D15 to D47, D20 to D48, D26 to D49, D23 to D5, D31 to D50, D36 to D51, D42 to D52, D47 to D53, D52 to D54, D57 to D55, D63 to D56, D74 to D57, D80 to D58, D5 to D59, D28 to D6, D16 to D60, D21 to D61, D27 to D62, D32 to D63, D37 to D64, D43 to D65, D48 to D66, D53 to D67, D58 to D68, D64 to D69, D33 to D7, D69 to D70, D75 to D71, D81 to D72, D6 to D73, D11 to D74, D22 to D75, D38 to D76, D59 to D77, D65 to D78, D70 to D79, D39 to D8, D76 to D80, D82 to D81, D44 to D9
Connections:
- net labels added: BATTERY_PIN, BLUE_LED, CC1, CC2, COL15, DATA+, DATA-, DCCH, EXT_VCC, POWER_PIN, PROG, RESET, Rotary-A, Rotary-B, SWC, SWD, VBAT, nRF_VDD
- net labels removed: +5V, D+, D-, DM-USB, DP-USB, GND-USB, MISO, MOSI, RGB, RST, SCK, VBUS-USB, VCC
- wire segments 506 -> 328
Other:
- note added: "LiPo Charging"
- note added: "Power & Filtering"
- moved on the sheet: D10, D11, D12, D13, D14, D6, D60, D61, D62, D63, D64, D65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

Commit message: updae
Parts:
- removed F1: 500mA, Fuse:Fuse_1206_3216Metric, symbol Device:Polyfuse_Small
- removed R1, R2: 5.1k, Resistor_SMD:R_0603_1608Metric, symbol Device:R_Small
- removed U1: USBLC6-2SC6, Package_TO_SOT_SMD:SOT-23-6, symbol Power_Protection:USBLC6-2SC6
- removed USB1: HRO-TYPE-C-31-M-12, Type-C:HRO-TYPE-C-31-M-12-HandSoldering, symbol keebio:HRO-TYPE-C-31-M-12
- added J4: RESET, random-keyboard-parts:PushButton_6x6mm_TH, symbol Connector_Generic:Conn_01x02
- J2: footprint Connector_PinHeader_2.54mm:PinHeader_1x02_P2.54mm_Vertical -> Connector_JST:JST_SH_BM02B-SRSS-TB_1x02-1MP_P1.00mm_Vertical
- J3: footprint nrfmicro:connector_usb -> Connector_JST:JST_SH_BM04B-SRSS-TB_1x04-1MP_P1.00mm_Vertical
- MX1, MX10, MX11, MX12, MX13, MX14, MX15, MX16, MX17, MX18, MX19, MX2, MX20, MX21, MX22, MX23, MX24, MX25, MX26, MX27, MX29, MX3, MX31, MX32, MX33, MX34, MX35, MX36, MX37, MX38, MX39, MX4, MX40, MX41, MX42, MX44, MX46, MX47, MX48, MX49, MX5, MX50, MX51, MX52, MX53, MX54, MX55, MX56, MX58, MX6, MX60, MX61, MX62, MX63, MX64, MX65, MX66, MX67, MX68, MX69, MX7, MX71, MX72, MX79, MX8, MX80, MX81, MX9: footprint MX_Only:MXOnly-1U-Hotswap -> MX_Only:MXOnly-1U-NoLED
- MX28: footprint MX_Only:MXOnly-2U-Hotswap -> MX_Only:MXOnly-2U-NoLED
- MX30, MX43: footprint MX_Only:MXOnly-1.5U-Hotswap -> MX_Only:MXOnly-1.5U-NoLED
- MX45, MX70: footprint MX_Only:MXOnly-1.75U-Hotswap -> MX_Only:MXOnly-1.75U-NoLED
- MX57, MX59: footprint MX_Only:MXOnly-2.25U-Hotswap -> MX_Only:MXOnly-2.25U-NoLED
- MX73, MX74, MX75, MX77, MX78: footprint MX_Only:MXOnly-1.25U-Hotswap -> MX_Only:MXOnly-1.25U-NoLED
- MX76: footprint MX_Only:MXOnly-6.25U-Hotswap-ReversedStabilizers -> MX_Only:MXOnly-6.25U-ReversedStabilizers-NoLED
Connections:
- net GND: now also J4.1 (Pin_1)
- net RESET: now also J4.2 (Pin_2)
- net ROW0: now also U2.35 (P0.24)
- net ROW1: now also U2.41 (P0.09/NFC1)
- net ROW2: now also U2.43 (P0.10/NFC2)
- net ROW3: now also U2.40 (P1.04)
- net ROW4: now also U2.42 (P1.06)
- net ROW5: now also U2.33 (P0.13)
- net SWC: now also J1.3 (Pin_3); no longer J1.4 (Pin_4)
- net SWD: now also J1.4 (Pin_4); no longer J1.3 (Pin_3)
- no-connect marks 2 -> 0
Other:
- moved on the sheet: J3

Commit message: big update and revision
Parts:
- added J5: Underglow, Connector_PinHeader_2.54mm:PinHeader_1x03_P2.54mm_Vertical, symbol Connector_Generic:Conn_01x03
- J4: footprint random-keyboard-parts:PushButton_6x6mm_TH -> random-keyboard-parts:SKQG-1155865
Connections:
- net COL0: now also U2.33 (P0.13)
- net COL1: now also U2.36 (P1.00)
- net COL10: now also MX78.1 (COL), U2.7 (P0.02/AIN0); no longer MX77.1 (COL)
- net COL11: now also U2.8 (P0.29/AIN5); no longer MX70.1 (COL), MX78.1 (COL)
- net COL12: now also MX70.1 (COL), U2.9 (P0.31/AIN7)
- net COL13: now also U2.10 (P0.30/AIN6)
- net COL14: now also U2.14 (P0.06)
- net COL15: now also U2.12 (P0.26)
- net COL2: now also U2.34 (P0.22)
- net COL3: now also U2.32 (P0.20)
- net COL4: now also U2.30 (P0.17)
- net COL5: now also U2.28 (P0.15)
- net COL6: now also U2.1 (P1.11)
- net COL7: now also U2.3 (P0.03/AIN1)
- net COL8: now also U2.4 (P0.28/AIN4)
- net COL9: now also MX77.1 (COL), U2.6 (P1.13)
- net GND: now also J5.1 (Pin_1)
- net ROW0: now also U2.38 (P1.02); no longer U2.35 (P0.24)
- net ROW2: now also U2.40 (P1.04); no longer U2.43 (P0.10/NFC2)
- net ROW3: now also U2.43 (P0.10/NFC2); no longer U2.40 (P1.04)
- net ROW5: now also U2.35 (P0.24); no longer U2.33 (P0.13)
- net Rotary-A: now also U2.20 (P0.12)
- net Rotary-B: now also U2.16 (P0.08)
- net VBUS: now also J5.3 (Pin_3)
- net RGB: now reaches U2.22 (P0.07)
- net RGB: now also J5.2 (Pin_2)
Other:
- moved on the sheet: D70, D77, D78, MX70, MX77, MX78, Y1
Changed lines of the file:
@@
 L MX_Alps_Hybrid:MX-NoLED MX70
 U 1 1 5E5C9E8C
-P 6600 5100
-F 0 "MX70" H 6633 5323 60  0000 C CNN
-F 1 "RShift" H 6633 5249 20  0000 C CNN
-F 2 "MX_Only:MXOnly-1.75U-NoLED" H 5975 5075 60  0001 C CNN
-F 3 "" H 5975 5075 60  0001 C CNN
-	1    6600 5100
+P 7100 5100
+F 0 "MX70" H 7133 5323 60  0000 C CNN
+F 1 "RShift" H 7133 5249 20  0000 C CNN
+F 2 "MX_Only:MXOnly-1.75U-NoLED" H 6475 5075 60  0001 C CNN
+F 3 "" H 6475 5075 60  0001 C CNN
+	1    7100 5100
 	1    0    0    -1
 $EndComp
@@
 L Diode:1N4148W D70
 U 1 1 5E5C9E92
-P 6500 5400
-F 0 "D70" V 6546 5320 50  0000 R CNN
-F 1 "1N4148W" V 6455 5320 50  0000 R CNN
-F 2 "master-Keebio-Parts:D_SOD-123-v2" H 6500 5225 50  0001 C CNN
-F 3 "https://www.vishay.com/docs/85748/1n4148w.pdf" H 6500 5400 50  0001 C CNN
-	1    6500 5400
-	0    -1   -1   0
-$EndComp
-Wire Wire Line
-	6550 5250 6500 5250
+P 7000 5400
+F 0 "D70" V 7046 5320 50  0000 R CNN
+F 1 "1N4148W" V 6955 5320 50  0000 R CNN
+F 2 "master-Keebio-Parts:D_SOD-123-v2" H 7000 5225 50  0001 C CNN
+F 3 "https://www.vishay.com/docs/85748/1n4148w.pdf" H 7000 5400 50  0001 C CNN
+	1    7000 5400
+	0    -1   -1   0
+$EndComp
+Wire Wire Line
+	7050 5250 7000 5250
 $Comp
 L MX_Alps_Hybrid:MX-NoLED MX71
@@
 L MX_Alps_Hybrid:MX-NoLED MX77
 U 1 1 5E5D954B
+P 5600 6100
+F 0 "MX77" H 5633 6323 60  0000 C CNN
+F 1 "RAlt" H 5633 6249 20  0000 C CNN
+F 2 "MX_Only:MXOnly-1.25U-NoLED" H 4975 6075 60  0001 C CNN
+F 3 "" H 4975 6075 60  0001 C CNN
+	1    5600 6100
+	1    0    0    -1
+$EndComp
+$Comp
+L Diode:1N4148W D77
+U 1 1 5E5D9551
+P 5500 6400
+F 0 "D77" V 5546 6320 50  0000 R CNN
+F 1 "1N4148W" V 5455 6320 50  0000 R CNN
+F 2 "master-Keebio-Parts:D_SOD-123-v2" H 5500 6225 50  0001 C CNN
+F 3 "https://www.vishay.com/docs/85748/1n4148w.pdf" H 5500 6400 50  0001 C CNN
+	1    5500 6400
+	0    -1   -1   0
+$EndComp
+Wire Wire Line
+	5550 6250 5500 6250
+$Comp
+L MX_Alps_Hybrid:MX-NoLED MX78
+U 1 1 5E5D9565
 P 6100 6100
-F 0 "MX77" H 6133 6323 60  0000 C CNN
-F 1 "RAlt" H 6133 6249 20  0000 C CNN
+F 0 "MX78" H 6133 6323 60  0000 C CNN
+F 1 "RCtrl" H 6133 6249 20  0000 C CNN
 F 2 "MX_Only:MXOnly-1.25U-NoLED" H 5475 6075 60  0001 C CNN
 F 3 "" H 5475 6075 60  0001 C CNN
@@
 $EndComp
 $Comp
-L Diode:1N4148W D77
-U 1 1 5E5D9551
+L Diode:1N4148W D78
+U 1 1 5E5D956B
 P 6000 6400
-F 0 "D77" V 6046 6320 50  0000 R CNN
+F 0 "D78" V 6046 6320 50  0000 R CNN
 F 1 "1N4148W" V 5955 6320 50  0000 R CNN
 F 2 "master-Keebio-Parts:D_SOD-123-v2" H 6000 6225 50  0001 C CNN
@@
 Wire Wire Line
 	6050 6250 6000 6250
-$Comp
-L MX_Alps_Hybrid:MX-NoLED MX78
-U 1 1 5E5D9565
-P 6600 6100
-F 0 "MX78" H 6633 6323 60  0000 C CNN
-F 1 "RCtrl" H 6633 6249 20  0000 C CNN
-F 2 "MX_Only:MXOnly-1.25U-NoLED" H 5975 6075 60  0001 C CNN
-F 3 "" H 5975 6075 60  0001 C CNN
-	1    6600 6100
-	1    0    0    -1
-$EndComp
-$Comp
-L Diode:1N4148W D78
-U 1 1 5E5D956B
-P 6500 6400
-F 0 "D78" V 6546 6320 50  0000 R CNN
-F 1 "1N4148W" V 6455 6320 50  0000 R CNN
-F 2 "master-Keebio-Parts:D_SOD-123-v2" H 6500 6225 50  0001 C CNN
-F 3 "https://www.vishay.com/docs/85748/1n4148w.pdf" H 6500 6400 50  0001 C CNN
-	1    6500 6400
-	0    -1   -1   0
-$EndComp
-Wire Wire Line
-	6550 6250 6500 6250
 $Comp
 L MX_Alps_Hybrid:MX-NoLED MX79
@@
 	6750 3050 6750 4050
 Connection ~ 6750 3050
-Connection ~ 6750 4050
-Wire Wire Line
-	6750 4050 6750 5050
-Connection ~ 6750 5050
-Wire Wire Line
-	6750 5050 6750 6050
+Wire Wire Line
+	5750 5050 5750 6050
 Wire Wire Line
 	7250 1050 7250 2050
@@
 Connection ~ 7250 3050
 Wire Wire Line
-	7250 3050 7250 6050
+	7250 3050 7250 5050
 Wire Wire Line
 	7750 1050 7750 2050
@@
 Wire Wire Line
 	6000 5550 5500 5550
-Connection ~ 6500 5550
-Wire Wire Line
-	6500 5550 6000 5550
 Connection ~ 7500 5550
 Wire Wire Line
-	7500 5550 6500 5550
+	7500 5550 7000 5550
 Wire Wire Line
 	1000 6550 1500 6550
@@
 Connection ~ 3500 6550
 Wire Wire Line
-	3500 6550 6000 6550
-Connection ~ 6000 6550
-Wire Wire Line
-	6000 6550 6500 6550
-Connection ~ 6500 6550
-Wire Wire Line
-	6500 6550 7000 6550
+	3500 6550 5500 6550
 Connection ~ 7000 6550
 Wire Wire Line
@@
 L power:GND #PWR09
 U 1 1 60680563
-P 1350 8050
-F 0 "#PWR09" H 1350 7800 50  0001 C CNN
-F 1 "GND" H 1355 7877 50  0000 C CNN
-F 2 "" H 1350 8050 50  0001 C CNN
-F 3 "" H 1350 8050 50  0001 C CNN
-	1    1350 8050
+P 1250 8050
+F 0 "#PWR09" H 1250 7800 50  0001 C CNN
+F 1 "GND" H 1255 7877 50  0000 C CNN
+F 2 "" H 1250 8050 50  0001 C CNN
+F 3 "" H 1250 8050 50  0001 C CNN
+	1    1250 8050
 	1    0    0    -1
 $EndComp
@@
 	3650 9650 3000 9650
 Wire Wire Line
-	1350 8050 1650 8050
+	1250 8050 1650 8050
 $Comp
 L Device:Crystal_Small Y1
 U 1 1 607CCB47
-P 1400 8750
-F 0 "Y1" V 1350 8450 50  0000 L CNN
-F 1 "32.768kHz" V 1450 8300 39  0000 L CNN
-F 2 "Crystal:Crystal_SMD_MicroCrystal_CM9V-T1A-2Pin_1.6x1.0mm" H 1400 8750 50  0001 C CNN
-F 3 "~" H 1400 8750 50  0001 C CNN
-	1    1400 8750
+P 1250 8750
+F 0 "Y1" V 1200 8450 50  0000 L CNN
+F 1 "32.768kHz" V 1300 8300 39  0000 L CNN
+F 2 "Crystal:Crystal_SMD_MicroCrystal_CM9V-T1A-2Pin_1.6x1.0mm" H 1250 8750 50  0001 C CNN
+F 3 "~" H 1250 8750 50  0001 C CNN
+	1    1250 8750
 	0    1    1    0
 $EndComp
 Wire Wire Line
-	1400 8650 1650 8650
-Wire Wire Line
-	1400 8850 1650 8850
+	1250 8650 1650 8650
+Wire Wire Line
+	1250 8850 1650 8850
 Text GLabel 1400 9050 0    50   Input ~ 0
 PROG
@@
 L power:GND #PWR012
 U 1 1 60861F51
-P 1400 9650
-F 0 "#PWR012" H 1400 9400 50  0001 C CNN
-F 1 "GND" H 1405 9477 50  0000 C CNN
-F 2 "" H 1400 9650 50  0001 C CNN
-F 3 "" H 1400 9650 50  0001 C CNN
-	1    1400 9650
-	1    0    0    -1
-$EndComp
-Wire Wire Line
-	1400 9650 1650 9650
+P 1300 9650
+F 0 "#PWR012" H 1300 9400 50  0001 C CNN
+F 1 "GND" H 1305 9477 50  0000 C CNN
+F 2 "" H 1300 9650 50  0001 C CNN
+F 3 "" H 1300 9650 50  0001 C CNN
+	1    1300 9650
+	1    0    0    -1
+$EndComp
+Wire Wire Line
+	1300 9650 1650 9650
 Text GLabel 1400 7750 0    50   Input ~ 0
 BLUE_LED
@@
 F 0 "J4" H 11530 4992 50  0000 L CNN
 F 1 "RESET" H 11530 4901 50  0000 L CNN
-F 2 "random-keyboard-parts:PushButton_6x6mm_TH" H 11450 5000 50  0001 C CNN
+F 2 "random-keyboard-parts:SKQG-1155865" H 11450 5000 50  0001 C CNN
 F 3 "~" H 11450 5000 50  0001 C CNN
 	1    11450 5000
@@
 	1    0    0    -1
 $EndComp
-Text GLabel 3000 8750 2    50   Input ~ 0
+Text GLabel 3000 8550 2    50   Input ~ 0
 ROW5
-Text GLabel 3000 8550 2    50   Input ~ 0
+Text GLabel 3000 8250 2    50   Input ~ 0
 ROW0
 Text GLabel 3000 7950 2    50   Input ~ 0
 ROW1
+Text GLabel 3000 8050 2    50   Input ~ 0
+ROW2
 Text GLabel 3000 7750 2    50   Input ~ 0
-ROW2
-Text GLabel 3000 8050 2    50   Input ~ 0
 ROW3
 Text GLabel 3000 7850 2    50   Input ~ 0
 ROW4
+Connection ~ 5500 6550
+Wire Wire Line
+	5500 6550 6000 6550
+Connection ~ 6000 6550
+Wire Wire Line
+	6000 6550 7000 6550
+Connection ~ 5750 5050
+Connection ~ 7000 5550
+Connection ~ 7250 5050
+Wire Wire Line
+	7250 5050 7250 6050
+Wire Wire Line
+	6000 5550 7000 5550
+Text GLabel 3000 8750 2    50   Input ~ 0
+COL0
+Text GLabel 3000 8450 2    50   Input ~ 0
+COL1
+Text GLabel 3000 8650 2    50   Input ~ 0
+COL2
+Text GLabel 3000 8850 2    50   Input ~ 0
+COL3
+Text GLabel 3000 9050 2    50   Input ~ 0
+COL4
+Text GLabel 3000 9250 2    50   Input ~ 0
+COL5
+Text GLabel 1650 7650 0    50   Input ~ 0
+COL6
+Text GLabel 1650 7850 0    50   Input ~ 0
+COL7
+Text GLabel 1650 7950 0    50   Input ~ 0
+COL8
+Text GLabel 1650 8150 0    50   Input ~ 0
+COL9
+Text GLabel 1650 8250 0    50   Input ~ 0
+COL10
+Text GLabel 1650 8350 0    50   Input ~ 0
+COL11
+Text GLabel 1650 8450 0    50   Input ~ 0
+COL12
+Text GLabel 1650 8550 0    50   Input ~ 0
+COL13
+Text GLabel 1650 8950 0    50   Input ~ 0
+COL14
+Text GLabel 1650 8750 0    50   Input ~ 0
+COL15
+Text GLabel 1650 9550 0    50   Input ~ 0
+Rotary-A
+Text GLabel 1650 9150 0    50   Input ~ 0
+Rotary-B
+$Comp
+L Connector_Generic:Conn_01x03 J5
+U 1 1 60F46879
+P 11450 5450
+F 0 "J5" H 11600 5400 50  0000 C CNN
+F 1 "Underglow" H 11750 5500 50  0000 C CNN
+F 2 "Connector_PinHeader_2.54mm:PinHeader_1x03_P2.54mm_Vertical" H 11450 5450 50  0001 C CNN
+F 3 "~" H 11450 5450 50  0001 C CNN
+	1    11450 5450
+	1    0    0    1
+$EndComp
+$Comp
+L power:GND #PWR0102
+U 1 1 60F48904
+P 11250 5550
+F 0 "#PWR0102" H 11250 5300 50  0001 C CNN
+F 1 "GND" H 11255 5377 50  0000 C CNN
+F 2 "" H 11250 5550 50  0001 C CNN
+F 3 "" H 11250 5550 50  0001 C CNN
+	1    11250 5550
+	1    0    0    -1
+$EndComp
+Text GLabel 11250 5350 0    39   Input ~ 0
+VBUS
+Text GLabel 11250 5450 0    50   Input ~ 0
+RGB
+Text GLabel 1650 9750 0    50   Input ~ 0
+RGB
 $EndSCHEMATC

Commit message: final
Parts:
- J5: footprint Connector_PinHeader_2.54mm:PinHeader_1x03_P2.54mm_Vertical -> Connector_PinHeader_2.00mm:PinHeader_1x03_P2.00mm_Vertical
Connections:
- net EXT_VCC: now also J5.3 (Pin_3)
- net VBUS: no longer J5.3 (Pin_3)
Changed lines of the file:
@@
 F 0 "J5" H 11600 5400 50  0000 C CNN
 F 1 "Underglow" H 11750 5500 50  0000 C CNN
-F 2 "Connector_PinHeader_2.54mm:PinHeader_1x03_P2.54mm_Vertical" H 11450 5450 50  0001 C CNN
+F 2 "Connector_PinHeader_2.00mm:PinHeader_1x03_P2.00mm_Vertical" H 11450 5450 50  0001 C CNN
 F 3 "~" H 11450 5450 50  0001 C CNN
 	1    11450 5450
@@
 	1    0    0    -1
 $EndComp
-Text GLabel 11250 5350 0    39   Input ~ 0
-VBUS
 Text GLabel 11250 5450 0    50   Input ~ 0
 RGB
 Text GLabel 1650 9750 0    50   Input ~ 0
 RGB
+Text GLabel 11250 5350 0    50   Input ~ 0
+EXT_VCC
 $EndSCHEMATC
