File: ridhaulakbar75.kicad_pcb (KiCad board)
At the start: 2 copper layers, 314.3 x 123.8 mm, 202 parts, among them J1 AVR-ISP-6, J2 Conn_01x04, U1 TEENSY2.0

Commit message: update
Parts:
- removed R1, R2: 5.1K, Resistor_SMD:R_0805_2012Metric_Pad1.15x1.40mm_HandSolder
- added C18: 0.1uF, Capacitor_SMD:C_0603_1608Metric_Pad1.05x0.95mm_HandSolder, B.Cu at (150.8, 243.7)
- added C9: 0.1uF, Capacitor_SMD:C_0603_1608Metric_Pad1.05x0.95mm_HandSolder, B.Cu at (133.3, 263.5)
- added LED18: WS2812B, WS2812B:WS2812B, B.Cu at (141.6, 232.3)
- added LED9: WS2812B, WS2812B:WS2812B, B.Cu at (157.2, 231.8)
- moved C1 287.9 mm to (73.8, 179.1), turned to 270 degrees
- moved C5 287.7 mm to (350.0, 102.7), turned to 90 degrees
- moved LED17 277.5 mm to (78.6, 102.7), turned to 90 degrees
- moved LED1 277.5 mm to (78.6, 179.1), turned to 270 degrees
- moved LED8 277.5 mm to (345.3, 179.1), turned to 270 degrees
- moved LED10 277.3 mm to (345.3, 102.7), turned to 90 degrees
- moved C17 268.7 mm to (83.3, 102.7), turned to 90 degrees
- moved C13 267.2 mm to (340.5, 179.1), turned to 270 degrees
- moved C10 215.4 mm to (111.9, 179.1), turned to 270 degrees
- moved C14 215.1 mm to (311.9, 102.7), turned to 90 degrees
- moved LED2 205.4 mm to (116.7, 179.1), turned to 270 degrees
- moved LED7 205.4 mm to (307.2, 179.1), turned to 270 degrees
- moved LED11 205.0 mm to (307.2, 102.7), turned to 90 degrees
- moved LED16 205.0 mm to (116.7, 102.7), turned to 90 degrees
- moved C4 195.4 mm to (302.4, 179.1), turned to 270 degrees
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- renumbered C2 to C10, C4 to C11, C6 to C12, C8 to C13, C10 to C14, C12 to C15, C14 to C16, C16 to C17, C3 to C2, C5 to C3, C7 to C4, C9 to C5, C11 to C6, C13 to C7, C15 to C8, D16 to D11, D11 to D12, D12 to D13, D13 to D14, D14 to D15, D15 to D16, D27 to D22, D22 to D23, D23 to D24, D24 to D25, D25 to D26, D26 to D27, D55 to D54, D56 to D55, D57 to D56, D58 to D57, D59 to D58, D54 to D59, D61 to D60, D62 to D61, D63 to D62, D64 to D63, D65 to D64, D66 to D65, D67 to D66, D68 to D67, D69 to D68, D71 to D69, D72 to D70, D73 to D71, D74 to D72, D75 to D73, D70 to D74, D76 to D75, D77 to D76, D78 to D77, D79 to D78, D80 to D79, D81 to D80, D82 to D81, D83 to D82, J2 to J1, J1 to J2, LED9 to LED10, LED10 to LED11, LED11 to LED12, LED12 to LED13, LED13 to LED14, LED14 to LED15, LED15 to LED16, LED16 to LED17, MX16 to MX11, MX11 to MX12, MX12 to MX13, MX13 to MX14, MX14 to MX15, MX15 to MX16, MX27 to MX22, MX22 to MX23, MX23 to MX24, MX24 to MX25, MX25 to MX26, MX26 to MX27, MX55 to MX54, MX56 to MX55, MX57 to MX56, MX58 to MX57, MX59 to MX58, MX54 to MX59, MX61 to MX60, MX62 to MX61, MX63 to MX62, MX64 to MX63, MX65 to MX64, MX66 to MX65, MX67 to MX66, MX68 to MX67, MX69 to MX68, MX71 to MX69, MX72 to MX70, MX73 to MX71, MX74 to MX72, MX75 to MX73, MX70 to MX74, MX76 to MX75, MX77 to MX76, MX78 to MX77, MX79 to MX78, MX80 to MX79, MX81 to MX80, MX82 to MX81, MX83 to MX82
Connections:
- J1 pad 1: VBUS-USB -> (no net)
- J1 pad 2: DM-USB -> (no net)
- J1 pad 3: DP-USB -> (no net)
- LED10 pad 4: Net-(LED8-Pad2) -> Net-(LED10-Pad4)
- LED17 pad 2: (no net) -> Net-(LED17-Pad2)
- USB1 pad 10: Net-(R2-Pad2) -> (no net)
- USB1 pad 11: VBUS-USB -> VBUS
- USB1 pad 2: VBUS-USB -> VBUS
- USB1 pad 4: Net-(R1-Pad2) -> (no net)
- USB1 pad 5: DM-USB -> D-
- USB1 pad 6: DP-USB -> D+
- USB1 pad 7: DM-USB -> D-
- USB1 pad 8: DP-USB -> D+
Routing:
- net +5V: track 0.00 -> 326.7 mm
- net ROW1: track 0.00 -> 224.6 mm
- net ROW0: track 0.00 -> 210.7 mm
- net Net-(D77-Pad2): track 0.00 -> 67.2 mm
- net Net-(D23-Pad2): track 0.00 -> 54.1 mm
- net Net-(D61-Pad2): track 0.00 -> 52.6 mm
- net Net-(D29-Pad2): track 0.00 -> 52.6 mm
- net Net-(D49-Pad2): track 0.00 -> 47.9 mm
- net Net-(D34-Pad2): track 0.00 -> 47.5 mm
- net Net-(D2-Pad2): track 0.00 -> 47.5 mm
- net Net-(D78-Pad2): track 0.00 -> 47.0 mm
- net Net-(LED11-Pad2): track 0.00 -> 45.3 mm
- net Net-(LED15-Pad2): track 0.00 -> 45.3 mm
- net Net-(LED14-Pad2): track 0.00 -> 45.3 mm
- net Net-(LED13-Pad2): track 0.00 -> 45.3 mm
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- added copper zone on B.Cu, net GND
Other:
- board text added: "D+"
- board text added: "D-"
- board text added: "G"
- board text added: "V"

Commit message: big update
Parts:
- removed C1, C10, C11, C12, C13, C14, C15, C16, C17, C18, C2, C3, C4, C5, C6, C7, C8, C9: 0.1uF, Capacitor_SMD:C_0603_1608Metric_Pad1.05x0.95mm_HandSolder
- removed the D71 at (301.2, 96.0)
- removed LED1, LED10, LED11, LED12, LED13, LED14, LED15, LED16, LED17, LED18, LED2, LED3, LED4, LED5, LED6, LED7, LED8, LED9: WS2812B, WS2812B:WS2812B
- removed the MX71 at (331.0, 90.5)
- added D83: 1N5819, Diode_SMD:D_SOD-323F, B.Cu at (146.6, 191.0)
- added F1: 500mA, Fuse:Fuse_1206_3216Metric, B.Cu at (209.5, 96.7)
- added J3: Ex_USB, nrfmicro:connector_usb, F.Cu at (203.3, 102.0)
- added LED: RED, LED_SMD:LED_0603_1608Metric, B.Cu at (151.5, 196.6)
- added LED: BLUE, LED_SMD:LED_0603_1608Metric, B.Cu at (151.5, 184.0)
- added Q1: AO3407, Package_TO_SOT_SMD:SOT-23, B.Cu at (146.7, 185.0)
- added Q2: AO3407, Package_TO_SOT_SMD:SOT-23, B.Cu at (146.7, 195.6)
- added R1: 5.1k, Resistor_SMD:R_0603_1608Metric, B.Cu at (200.0, 82.5)
- added R2: 5.1k, Resistor_SMD:R_0603_1608Metric, B.Cu at (214.3, 82.5)
- added R3: 820K, Resistor_SMD:R_0603_1608Metric, B.Cu at (155.1, 184.6)
- added R4: 1K, Resistor_SMD:R_0603_1608Metric, B.Cu at (151.6, 185.7)
- added R5: 2M, Resistor_SMD:R_0603_1608Metric, B.Cu at (155.1, 188.0)
- added R6: 2M, Resistor_SMD:R_0603_1608Metric, B.Cu at (146.5, 192.9)
- added R7: 100k, Resistor_SMD:R_0603_1608Metric, B.Cu at (145.7, 188.3)
- added R8: 1K, Resistor_SMD:R_0603_1608Metric, B.Cu at (151.6, 194.8)
- added R9: 2K, Resistor_SMD:R_0603_1608Metric, B.Cu at (155.1, 192.4)
- added SW1: Rotary_Encoder_Switch, master-Keebio-Parts:RotaryEncoder_EC11-no-legs, B.Cu at (350.0, 90.2)
- added U2: E73-2G4M08S1C-52840, nrfmicro:E73-2G4M08S1C-52840, B.Cu at (156.5, 190.4)
- added U3: XC6220B331MR, Package_TO_SOT_SMD:SOT-23-5, B.Cu at (151.1, 188.4)
- added U4: TP4054, Package_TO_SOT_SMD:SOT-23-5, B.Cu at (151.1, 192.1)
- added Y1: 32.768kHz, Crystal:Crystal_SMD_MicroCrystal_CM9V-T1A-2Pin_1.6x1.0mm, B.Cu at (154.9, 196.1)
- J1: value Conn_01x04 -> SWD; footprint Connector_PinHeader_2.54mm:PinHeader_1x04_P2.54mm_Vertical -> nrfmicro:connector_swd
- J2: value AVR-ISP-6 -> Ex_Bat; footprint random-keyboard-parts:Reset_Pretty-Mask -> Connector_PinHeader_2.54mm:PinHeader_1x02_P2.54mm_Vertical
- MX1, MX18: footprint MX_Only:MXOnly-1U-NoLED -> MX_Only:MXOnly-1U-Hotswap
- MX10: renamed from MX49; footprint MX_Only:MXOnly-1U-NoLED -> MX_Only:MXOnly-1U-Hotswap
- MX11: renamed from MX54; footprint MX_Only:MXOnly-1U-NoLED -> MX_Only:MXOnly-1U-Hotswap
- MX12: renamed from MX60; footprint MX_Only:MXOnly-1U-NoLED -> MX_Only:MXOnly-1U-Hotswap
- MX13: renamed from MX66; footprint MX_Only:MXOnly-1U-NoLED -> MX_Only:MXOnly-1U-Hotswap
- MX14: renamed from MX77; footprint MX_Only:MXOnly-1U-NoLED -> MX_Only:MXOnly-1U-Hotswap
- MX15: renamed from MX2; footprint MX_Only:MXOnly-1U-NoLED -> MX_Only:MXOnly-1U-Hotswap
- MX16: renamed from MX8; footprint MX_Only:MXOnly-1U-NoLED -> MX_Only:MXOnly-1U-Hotswap
- MX17: renamed from MX13; footprint MX_Only:MXOnly-1U-NoLED -> MX_Only:MXOnly-1U-Hotswap
- MX19: renamed from MX24; footprint MX_Only:MXOnly-1U-NoLED -> MX_Only:MXOnly-1U-Hotswap
- MX2: renamed from MX7; footprint MX_Only:MXOnly-1U-NoLED -> MX_Only:MXOnly-1U-Hotswap
- MX20: renamed from MX29; footprint MX_Only:MXOnly-1U-NoLED -> MX_Only:MXOnly-1U-Hotswap
- MX21: renamed from MX34; footprint MX_Only:MXOnly-1U-NoLED -> MX_Only:MXOnly-1U-Hotswap
- MX22: renamed from MX40; footprint MX_Only:MXOnly-1U-NoLED -> MX_Only:MXOnly-1U-Hotswap
- MX23: renamed from MX45; footprint MX_Only:MXOnly-1U-NoLED -> MX_Only:MXOnly-1U-Hotswap
- MX24: renamed from MX50; footprint MX_Only:MXOnly-1U-NoLED -> MX_Only:MXOnly-1U-Hotswap
- MX25: renamed from MX55; footprint MX_Only:MXOnly-1U-NoLED -> MX_Only:MXOnly-1U-Hotswap
- MX26: renamed from MX61; footprint MX_Only:MXOnly-1U-NoLED -> MX_Only:MXOnly-1U-Hotswap
- MX27: renamed from MX67; footprint MX_Only:MXOnly-1U-NoLED -> MX_Only:MXOnly-1U-Hotswap
- MX28: renamed from MX72; footprint MX_Only:MXOnly-2U-NoLED -> MX_Only:MXOnly-2U-Hotswap
- MX29: renamed from MX78; footprint MX_Only:MXOnly-1U-NoLED -> MX_Only:MXOnly-1U-Hotswap
- MX3: renamed from MX12; footprint MX_Only:MXOnly-1U-NoLED -> MX_Only:MXOnly-1U-Hotswap
- MX30: renamed from MX3; footprint MX_Only:MXOnly-1.5U-NoLED -> MX_Only:MXOnly-1.5U-Hotswap
- MX31: renamed from MX9; footprint MX_Only:MXOnly-1U-NoLED -> MX_Only:MXOnly-1U-Hotswap
- MX32: renamed from MX14; footprint MX_Only:MXOnly-1U-NoLED -> MX_Only:MXOnly-1U-Hotswap
- MX33: renamed from MX19; footprint MX_Only:MXOnly-1U-NoLED -> MX_Only:MXOnly-1U-Hotswap
- MX34: renamed from MX25; footprint MX_Only:MXOnly-1U-NoLED -> MX_Only:MXOnly-1U-Hotswap
- MX35: renamed from MX30; footprint MX_Only:MXOnly-1U-NoLED -> MX_Only:MXOnly-1U-Hotswap
- MX36: renamed from MX35; footprint MX_Only:MXOnly-1U-NoLED -> MX_Only:MXOnly-1U-Hotswap
- MX37: renamed from MX41; footprint MX_Only:MXOnly-1U-NoLED -> MX_Only:MXOnly-1U-Hotswap
- MX38: renamed from MX46; footprint MX_Only:MXOnly-1U-NoLED -> MX_Only:MXOnly-1U-Hotswap
- MX39: renamed from MX51; footprint MX_Only:MXOnly-1U-NoLED -> MX_Only:MXOnly-1U-Hotswap
- MX4: renamed from MX17; footprint MX_Only:MXOnly-1U-NoLED -> MX_Only:MXOnly-1U-Hotswap
- MX40: renamed from MX56; footprint MX_Only:MXOnly-1U-NoLED -> MX_Only:MXOnly-1U-Hotswap
- MX41: renamed from MX62; footprint MX_Only:MXOnly-1U-NoLED -> MX_Only:MXOnly-1U-Hotswap
- MX42: renamed from MX68; footprint MX_Only:MXOnly-1U-NoLED -> MX_Only:MXOnly-1U-Hotswap
- MX43: renamed from MX73; footprint MX_Only:MXOnly-1.5U-NoLED -> MX_Only:MXOnly-1.5U-Hotswap
- MX44: renamed from MX79; footprint MX_Only:MXOnly-1U-NoLED -> MX_Only:MXOnly-1U-Hotswap
- MX45: renamed from MX4; footprint MX_Only:MXOnly-1.75U-NoLED -> MX_Only:MXOnly-1.75U-Hotswap
- MX46: renamed from MX10; footprint MX_Only:MXOnly-1U-NoLED -> MX_Only:MXOnly-1U-Hotswap
- MX47: renamed from MX15; footprint MX_Only:MXOnly-1U-NoLED -> MX_Only:MXOnly-1U-Hotswap
- MX48: renamed from MX20; footprint MX_Only:MXOnly-1U-NoLED -> MX_Only:MXOnly-1U-Hotswap
- MX49: renamed from MX26; footprint MX_Only:MXOnly-1U-NoLED -> MX_Only:MXOnly-1U-Hotswap
- MX5: renamed from MX23; footprint MX_Only:MXOnly-1U-NoLED -> MX_Only:MXOnly-1U-Hotswap
- MX50: renamed from MX31; footprint MX_Only:MXOnly-1U-NoLED -> MX_Only:MXOnly-1U-Hotswap
- MX51: renamed from MX36; footprint MX_Only:MXOnly-1U-NoLED -> MX_Only:MXOnly-1U-Hotswap
- MX52: renamed from MX42; footprint MX_Only:MXOnly-1U-NoLED -> MX_Only:MXOnly-1U-Hotswap
- MX53: renamed from MX47; footprint MX_Only:MXOnly-1U-NoLED -> MX_Only:MXOnly-1U-Hotswap
- MX54: renamed from MX52; footprint MX_Only:MXOnly-1U-NoLED -> MX_Only:MXOnly-1U-Hotswap
- MX55: renamed from MX57; footprint MX_Only:MXOnly-1U-NoLED -> MX_Only:MXOnly-1U-Hotswap
- MX56: renamed from MX63; footprint MX_Only:MXOnly-1U-NoLED -> MX_Only:MXOnly-1U-Hotswap
- MX57: renamed from MX74; footprint MX_Only:MXOnly-2.25U-NoLED -> MX_Only:MXOnly-2.25U-Hotswap
- MX58: renamed from MX80; footprint MX_Only:MXOnly-1U-NoLED -> MX_Only:MXOnly-1U-Hotswap
- MX59: renamed from MX5; footprint MX_Only:MXOnly-2.25U-NoLED -> MX_Only:MXOnly-2.25U-Hotswap
- MX6: renamed from MX28; footprint MX_Only:MXOnly-1U-NoLED -> MX_Only:MXOnly-1U-Hotswap
- MX60: renamed from MX16; footprint MX_Only:MXOnly-1U-NoLED -> MX_Only:MXOnly-1U-Hotswap
- MX61: renamed from MX21; footprint MX_Only:MXOnly-1U-NoLED -> MX_Only:MXOnly-1U-Hotswap
- MX62: renamed from MX27; footprint MX_Only:MXOnly-1U-NoLED -> MX_Only:MXOnly-1U-Hotswap
- MX63: renamed from MX32; footprint MX_Only:MXOnly-1U-NoLED -> MX_Only:MXOnly-1U-Hotswap
- MX64: renamed from MX37; footprint MX_Only:MXOnly-1U-NoLED -> MX_Only:MXOnly-1U-Hotswap
- MX65: renamed from MX43; footprint MX_Only:MXOnly-1U-NoLED -> MX_Only:MXOnly-1U-Hotswap
- MX66: renamed from MX48; footprint MX_Only:MXOnly-1U-NoLED -> MX_Only:MXOnly-1U-Hotswap
- MX67: renamed from MX53; footprint MX_Only:MXOnly-1U-NoLED -> MX_Only:MXOnly-1U-Hotswap
- MX68: renamed from MX58; footprint MX_Only:MXOnly-1U-NoLED -> MX_Only:MXOnly-1U-Hotswap
- MX69: renamed from MX64; footprint MX_Only:MXOnly-1U-NoLED -> MX_Only:MXOnly-1U-Hotswap
- MX7: renamed from MX33; footprint MX_Only:MXOnly-1U-NoLED -> MX_Only:MXOnly-1U-Hotswap
- MX70: renamed from MX69; footprint MX_Only:MXOnly-1.75U-NoLED -> MX_Only:MXOnly-1.75U-Hotswap
- MX71: renamed from MX75; footprint MX_Only:MXOnly-1U-NoLED -> MX_Only:MXOnly-1U-Hotswap
- MX72: renamed from MX81; footprint MX_Only:MXOnly-1U-NoLED -> MX_Only:MXOnly-1U-Hotswap
- MX73: renamed from MX6; footprint MX_Only:MXOnly-1.5U-NoLED -> MX_Only:MXOnly-1.25U-Hotswap
- MX74: renamed from MX11; footprint MX_Only:MXOnly-1U-NoLED -> MX_Only:MXOnly-1.25U-Hotswap
- MX75: renamed from MX22; footprint MX_Only:MXOnly-1.5U-NoLED -> MX_Only:MXOnly-1.25U-Hotswap
- MX76: renamed from MX38; footprint MX_Only:MXOnly-7U-NoLED -> MX_Only:MXOnly-6.25U-Hotswap-ReversedStabilizers
- MX77: renamed from MX59; footprint MX_Only:MXOnly-1U-NoLED -> MX_Only:MXOnly-1.25U-Hotswap
- MX78: renamed from MX65; footprint MX_Only:MXOnly-1U-NoLED -> MX_Only:MXOnly-1.25U-Hotswap
- MX79: renamed from MX70; footprint MX_Only:MXOnly-1U-NoLED -> MX_Only:MXOnly-1U-Hotswap
- MX8: renamed from MX39; footprint MX_Only:MXOnly-1U-NoLED -> MX_Only:MXOnly-1U-Hotswap
- MX80: renamed from MX76; footprint MX_Only:MXOnly-1U-NoLED -> MX_Only:MXOnly-1U-Hotswap
- MX81: renamed from MX82; footprint MX_Only:MXOnly-1U-NoLED -> MX_Only:MXOnly-1U-Hotswap
- MX9: renamed from MX44; footprint MX_Only:MXOnly-1U-NoLED -> MX_Only:MXOnly-1U-Hotswap
- U1: value TEENSY2.0 -> USBLC6-2SC6; footprint master-Keebio-Parts:Teensy_2.0 -> Package_TO_SOT_SMD:SOT-23-6
- USB1: footprint master-Keebio-Parts:HRO-TYPE-C-31-M-12-Assembly -> Type-C:HRO-TYPE-C-31-M-12-HandSoldering
- moved J1 142.1 mm to (170.2, 190.4), turned to 90 degrees
- moved USB1 131.2 mm to (207.2, 73.0)
- moved J2 126.8 mm to (162.7, 84.1), turned to 270 degrees
- moved U1 98.3 mm to (205.3, 97.2)
- moved D5 56.1 mm to (158.4, 97.7)
- moved D14 53.5 mm to (357.1, 97.7)
- moved D26 49.7 mm to (282.3, 121.5)
- moved D20 49.7 mm to (168.0, 121.5)
- moved D35 49.7 mm to (177.5, 140.6)
- moved D41 49.7 mm to (291.8, 140.6)
- moved D50 49.7 mm to (182.3, 159.6)
- moved D56 49.7 mm to (296.6, 159.6)
- moved D73 47.1 mm to (77.5, 196.1)
- moved D9 43.0 mm to (244.2, 97.7)
- moved D4 39.4 mm to (139.4, 97.7)
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- renumbered D49 to D10, D54 to D11, D60 to D12, D66 to D13, D77 to D14, D2 to D15, D8 to D16, D13 to D17, D24 to D19, D7 to D2, D29 to D20, D34 to D21, D40 to D22, D45 to D23, D50 to D24, D55 to D25, D61 to D26, D67 to D27, D72 to D28, D78 to D29, D12 to D3, D3 to D30, D9 to D31, D14 to D32, D19 to D33, D25 to D34, D30 to D35, D35 to D36, D41 to D37, D46 to D38, D51 to D39, D17 to D4, D56 to D40, D62 to D41, D68 to D42, D73 to D43, D79 to D44, D4 to D45, D10 to D46, D15 to D47, D20 to D48, D26 to D49, D23 to D5, D31 to D50, D36 to D51, D42 to D52, D47 to D53, D52 to D54, D57 to D55, D63 to D56, D74 to D57, D80 to D58, D5 to D59, D28 to D6, D16 to D60, D21 to D61, D27 to D62, D32 to D63, D37 to D64, D43 to D65, D48 to D66, D53 to D67, D58 to D68, D64 to D69, D33 to D7, D69 to D70, D75 to D71, D81 to D72, D6 to D73, D11 to D74, D22 to D75, D38 to D76, D59 to D77, D65 to D78, D70 to D79, D39 to D8, D76 to D80, D82 to D81, D44 to D9
Connections:
- J1 pad 1: (no net) -> nRF_VDD
- J1 pad 2: (no net) -> GND
- J1 pad 3: (no net) -> SWD
- J1 pad 4: GND-USB -> SWC
- J2 pad 1: MISO -> GND
- J2 pad 2: VCC -> VBAT
- MX10 pad 1: COL9 -> COL11
- MX11 pad 1: COL10 -> COL12
- MX12 pad 1: COL11 -> COL13
- MX13 pad 1: COL12 -> COL14
- MX14 pad 1: COL14 -> COL15
- MX6 pad 1: COL5 -> COL6
- MX60 pad 1: COL2 -> COL1
- MX61 pad 1: COL3 -> COL2
- MX62 pad 1: COL4 -> COL3
- MX63 pad 1: COL5 -> COL4
- MX64 pad 1: COL6 -> COL5
- MX65 pad 1: COL7 -> COL6
- MX66 pad 1: COL8 -> COL7
- MX67 pad 1: COL9 -> COL8
- MX68 pad 1: COL10 -> COL9
- MX69 pad 1: COL11 -> COL10
- MX7 pad 1: COL6 -> COL7
- MX70 pad 1: COL12 -> COL11
- MX75 pad 1: COL3 -> COL2
- MX76 pad 1: COL6 -> COL5
- MX8 pad 1: COL7 -> COL8
- MX9 pad 1: COL8 -> COL9
- U1 pad 1: GND -> Net-(U1-Pad1)
- U1 pad 2: ROW0 -> GND
- U1 pad 3: SCK -> Net-(U1-Pad3)
- U1 pad 4: MOSI -> DATA-
- U1 pad 5: MISO -> Net-(F1-Pad1)
- U1 pad 6: COL0 -> DATA+
- USB1 pad 1: GND-USB -> GND
- USB1 pad 10: (no net) -> CC2
- USB1 pad 11: VBUS -> Net-(F1-Pad1)
- USB1 pad 12: GND-USB -> GND
- USB1 pad 13: GND-USB -> GND
- USB1 pad 2: VBUS -> Net-(F1-Pad1)
- USB1 pad 4: (no net) -> CC1
- USB1 pad 5: D- -> Net-(U1-Pad3)
- USB1 pad 6: D+ -> Net-(U1-Pad1)
- USB1 pad 7: D- -> Net-(U1-Pad3)
- USB1 pad 8: D+ -> Net-(U1-Pad1)
Routing:
- net +5V: track 326.7 -> 0.00 mm
- net ROW1: track 224.6 -> 0.00 mm
- net VBUS: track 0.00 -> 213.1 mm, vias 0 -> 6
- net ROW0: track 210.7 -> 0.00 mm
- net DATA-: track 0.00 -> 133.5 mm, vias 0 -> 2
- net DATA+: track 0.00 -> 126.4 mm, vias 0 -> 2
- net GND: track 0.00 -> 81.0 mm, vias 0 -> 8
- net Net-(D5-Pad2): track 54.1 -> 0.00 mm
- net Net-(D26-Pad2): track 52.6 -> 0.00 mm
- net Net-(D20-Pad2): track 52.6 -> 0.00 mm
- net Net-(D14-Pad2): track 67.2 -> 16.5 mm
- net Net-(D21-Pad2): track 47.5 -> 0.00 mm
- net Net-(D15-Pad2): track 47.5 -> 0.00 mm
- net Net-(D29-Pad2): track 47.0 -> 0.00 mm
- net Net-(LED11-Pad2): track 45.3 -> 0.00 mm
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- removed copper zone on B.Cu, net GND
Other:
- board size 314.3 x 123.8 mm -> 304.8 x 127 mm
- board text removed: "D+"
- board text removed: "D-"
- board text removed: "G"
- board text removed: "V"

Commit message: updae
Parts:
- removed F1: 500mA, Fuse:Fuse_1206_3216Metric
- removed R1, R2: 5.1k, Resistor_SMD:R_0603_1608Metric
- removed U1: USBLC6-2SC6, Package_TO_SOT_SMD:SOT-23-6
- removed USB1: HRO-TYPE-C-31-M-12, Type-C:HRO-TYPE-C-31-M-12-HandSoldering
- added J4: RESET, random-keyboard-parts:PushButton_6x6mm_TH, B.Cu at (212.5, 193.8)
- J1: moved to F.Cu
- J2: footprint Connector_PinHeader_2.54mm:PinHeader_1x02_P2.54mm_Vertical -> Connector_JST:JST_SH_BM02B-SRSS-TB_1x02-1MP_P1.00mm_Vertical
- J3: footprint nrfmicro:connector_usb -> Connector_JST:JST_SH_BM04B-SRSS-TB_1x04-1MP_P1.00mm_Vertical; moved to B.Cu
- MX1, MX10, MX11, MX12, MX13, MX14, MX15, MX16, MX17, MX18, MX19, MX2, MX20, MX21, MX22, MX23, MX24, MX25, MX26, MX27, MX29, MX3, MX31, MX32, MX33, MX34, MX35, MX36, MX37, MX38, MX39, MX4, MX40, MX41, MX42, MX44, MX46, MX47, MX48, MX49, MX5, MX50, MX51, MX52, MX53, MX54, MX55, MX56, MX58, MX6, MX60, MX61, MX62, MX63, MX64, MX65, MX66, MX67, MX68, MX69, MX7, MX71, MX72, MX79, MX8, MX80, MX81, MX9: footprint MX_Only:MXOnly-1U-Hotswap -> MX_Only:MXOnly-1U-NoLED
- MX28: footprint MX_Only:MXOnly-2U-Hotswap -> MX_Only:MXOnly-2U-NoLED
- MX30, MX43: footprint MX_Only:MXOnly-1.5U-Hotswap -> MX_Only:MXOnly-1.5U-NoLED
- MX45, MX70: footprint MX_Only:MXOnly-1.75U-Hotswap -> MX_Only:MXOnly-1.75U-NoLED
- MX57, MX59: footprint MX_Only:MXOnly-2.25U-Hotswap -> MX_Only:MXOnly-2.25U-NoLED
- MX73, MX74, MX75, MX77, MX78: footprint MX_Only:MXOnly-1.25U-Hotswap -> MX_Only:MXOnly-1.25U-NoLED
- MX76: footprint MX_Only:MXOnly-6.25U-Hotswap-ReversedStabilizers -> MX_Only:MXOnly-6.25U-ReversedStabilizers-NoLED
- moved J2 121.2 mm to (221.5, 190.2), turned to 180 degrees
- moved J3 88.2 mm to (202.4, 190.2), turned to 180 degrees
- moved R7 27.8 mm to (173.5, 186.3), turned to 0 degrees
- moved J1 23.5 mm to (146.7, 190.5)
- moved R4 22.7 mm to (173.5, 191.3)
- moved D82 22.5 mm to (173.5, 189.0)
- moved D83 22.4 mm to (168.3, 185.4), turned to 90 degrees
- moved D84 22.1 mm to (173.5, 194.1)
- moved R8 22.0 mm to (173.5, 196.4)
- moved Q1 19.4 mm to (165.5, 189.9), turned to 90 degrees
- moved R6 19.3 mm to (165.7, 192.7), turned to 180 degrees
- moved Q2 18.8 mm to (165.5, 195.5), turned to 270 degrees
- moved U4 18.7 mm to (169.5, 195.3), turned to 90 degrees
- moved U3 18.5 mm to (169.5, 190.2), turned to 90 degrees
- moved R9 17.0 mm to (170.6, 185.6)
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- renumbered LED to D82, LED to D84
Connections:
- J1 pad 3: SWD -> SWC
- J1 pad 4: SWC -> SWD
- U2 pad 26: (no net) -> RESET
- U2 pad 33: (no net) -> ROW5
- U2 pad 35: (no net) -> ROW0
- U2 pad 40: (no net) -> ROW3
- U2 pad 41: (no net) -> ROW1
- U2 pad 42: (no net) -> ROW4
- U2 pad 43: (no net) -> ROW2
Routing:
- net VBUS: track 213.1 -> 62.7 mm, vias 6 -> 2
- net DATA-: track 133.5 -> 54.0 mm, vias 2 -> 0
- net DATA+: track 126.4 -> 56.9 mm, vias 2 -> 0
- net RESET: track 0.00 -> 60.0 mm, vias 0 -> 1
- net GND: track 81.0 -> 133.0 mm, vias 8 -> 6
- net VBAT: track 22.0 -> 65.9 mm, vias 3 -> 2
- net Net-(F1-Pad1): track 33.1 -> 0.00 mm, vias 2 -> 0
- net Net-(U1-Pad1): track 22.8 -> 0.00 mm
- net Net-(U1-Pad3): track 20.2 -> 0.00 mm
- net POWER_PIN: track 26.1 -> 9.33 mm, vias 2 -> 0
- net nRF_VDD: track 17.7 -> 32.3 mm
- net Net-(D14-Pad2): track 16.5 -> 2.19 mm
- net Net-(D13-Pad2): track 11.7 -> 0.00 mm
- net Net-(D12-Pad2): track 11.7 -> 0.00 mm
- net Net-(D9-Pad2): track 11.7 -> 0.00 mm
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Other:
- board size 304.8 x 127 mm -> 304.8 x 119.1 mm

Commit message: big update and revision
Parts:
- added J5: Underglow, Connector_PinHeader_2.54mm:PinHeader_1x03_P2.54mm_Vertical, B.Cu at (214.5, 208.0)
- J4: footprint random-keyboard-parts:PushButton_6x6mm_TH -> random-keyboard-parts:SKQG-1155865
- moved J4 13.0 mm to (205.2, 204.6)
- moved D61 6.24 mm to (134.6, 173.0)
- moved D72 6.12 mm to (358.1, 173.0)
- moved D29 6.12 mm to (358.1, 115.8)
- moved D44 6.12 mm to (358.1, 134.9)
- moved D58 6.12 mm to (358.1, 153.9)
- moved D14 5.81 mm to (358.1, 92.0)
- moved D59 5.72 mm to (96.5, 173.0)
- moved D60 5.72 mm to (115.6, 173.0)
- moved D62 5.72 mm to (153.7, 173.0)
- moved D63 5.72 mm to (172.7, 173.0)
- moved D64 5.72 mm to (191.8, 173.0)
- moved D65 5.72 mm to (210.8, 173.0)
- moved D66 5.72 mm to (229.9, 173.0)
- moved D67 5.72 mm to (248.9, 173.0)
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Connections:
- MX70 pad 1: COL11 -> COL12
- MX77 pad 1: COL10 -> COL9
- MX78 pad 1: COL11 -> COL10
- SW1 pad A: (no net) -> Rotary-A
- SW1 pad B: (no net) -> Rotary-B
- U2 pad 1: (no net) -> COL6
- U2 pad 10: (no net) -> COL13
- U2 pad 12: (no net) -> COL15
- U2 pad 14: (no net) -> COL14
- U2 pad 16: (no net) -> Rotary-B
- U2 pad 20: (no net) -> Rotary-A
- U2 pad 22: (no net) -> RGB
- U2 pad 28: (no net) -> COL5
- U2 pad 3: (no net) -> COL7
- U2 pad 30: (no net) -> COL4
- U2 pad 32: (no net) -> COL3
- U2 pad 33: ROW5 -> COL0
- U2 pad 34: (no net) -> COL2
- U2 pad 35: ROW0 -> ROW5
- U2 pad 36: (no net) -> COL1
- U2 pad 38: (no net) -> ROW0
- U2 pad 4: (no net) -> COL8
- U2 pad 40: ROW3 -> ROW2
- U2 pad 43: ROW2 -> ROW3
- U2 pad 6: (no net) -> COL9
- U2 pad 7: (no net) -> COL10
- U2 pad 8: (no net) -> COL11
- U2 pad 9: (no net) -> COL12
Routing:
- net ROW0: track 0.00 -> 497.3 mm
- net ROW1: track 0.00 -> 468.9 mm
- net ROW2: track 0.00 -> 450.4 mm
- net ROW3: track 0.00 -> 426.8 mm
- net ROW4: track 0.00 -> 334.5 mm
- net COL14: track 0.00 -> 311.0 mm, vias 0 -> 2
- net COL13: track 0.00 -> 293.0 mm, vias 0 -> 2
- net ROW5: track 0.00 -> 289.3 mm
- net COL15: track 0.00 -> 287.3 mm
- net Rotary-B: track 0.00 -> 286.1 mm
- net Rotary-A: track 0.00 -> 285.8 mm
- net COL12: track 0.00 -> 259.8 mm, vias 0 -> 2
- net COL11: track 0.00 -> 233.1 mm, vias 0 -> 1
- net COL9: track 0.00 -> 218.0 mm, vias 0 -> 2
- net COL10: track 0.00 -> 211.6 mm, vias 0 -> 2
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
Commit message: final
Parts:
- added G***: LOGO, locallib:logo c, F.Cu at (235.7, 190.2)
- added REF**: 7U, MX_Only:MXOnly-7U-ReversedStabilizers-NoLED, F.Cu at (197.6, 190.5)
- added REF**: 1.5U, MX_Only:MXOnly-1.5U-NoLED, F.Cu at (278.6, 190.5)
- added REF**: 1.5U, MX_Only:MXOnly-1.5U-NoLED, F.Cu at (116.7, 190.5)
- added REF**: Stepped, MX_Only:MXOnly-1.25U-NoLED, F.Cu at (66.7, 152.4)
- added REF**: 1U, MX_Only:MXOnly-1U-NoLED, F.Cu at (92.9, 190.5)
- added REF**: 1.5U, MX_Only:MXOnly-1.5U-NoLED, F.Cu at (69.1, 190.5)
- RGB: renamed from J5; footprint Connector_PinHeader_2.54mm:PinHeader_1x03_P2.54mm_Vertical -> Connector_PinHeader_2.00mm:PinHeader_1x03_P2.00mm_Vertical
- moved USB 25.3 mm to (227.7, 189.6)
- moved RGB 19.6 mm to (215.7, 188.4), turned to 270 degrees
- moved RESET 15.8 mm to (217.7, 194.8), turned to 0 degrees
- moved BATT 12.8 mm to (208.6, 189.6)
- renumbered J2 to BATT, J4 to RESET, J3 to USB
Connections:
- Q1 pad 3: (no net) -> EXT_VCC
- RGB pad 3: VBUS -> EXT_VCC
Routing:
- net DATA+: track 0.09 -> 82.7 mm
- net DATA-: track 0.00 -> 80.3 mm
- net RGB: track 0.00 -> 75.8 mm
- net EXT_VCC: track 0.00 -> 59.4 mm, vias 0 -> 1
- net GND: track 100.9 -> 155.7 mm, vias 7 -> 8
- net RESET: track 10.1 -> 58.8 mm
- net VBUS: track 60.7 -> 90.8 mm
- net VBAT: track 40.2 -> 53.7 mm
- net COL4: track 149.7 -> 139.8 mm
- net COL0: track 208.8 -> 214.0 mm
- net Rotary-B: track 286.1 -> 291.2 mm
- net Net-(D45-Pad2): track 15.1 -> 19.8 mm
- net COL2: track 169.5 -> 165.9 mm
- net Rotary-A: track 285.8 -> 289.0 mm
- net COL5: track 151.7 -> 154.2 mm
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- added copper zone on B.Cu, net GND
- added copper zone on F.Cu, net GND
Other:
- board text added: "G D+ D- V"
- board text added: "G V"
- board text added: "V D G"

Commit message: add usb c back and add iso
Parts:
- added F1: 500mA, Fuse:Fuse_1206_3216Metric, B.Cu at (210.2, 99.9)
- added R1: 5.1K, Resistor_SMD:R_0603_1608Metric, B.Cu at (197.6, 82.5)
- added R2: 5.1K, Resistor_SMD:R_0603_1608Metric, B.Cu at (216.7, 82.5)
- added REF**: 1U, MX_Only:MXOnly-1U-NoLED, F.Cu at (307.2, 152.4)
- added REF**: ISO, MX_Only:MXOnly-ISO-ReversedStabilizers, F.Cu at (328.6, 142.9)
- added U1: USBLC6-2SC6, Package_TO_SOT_SMD:SOT-23-6, B.Cu at (205.4, 99.9)
- added USB1: HRO-TYPE-C-31-M-12, Type-C:HRO-TYPE-C-31-M-12-HandSoldering, B.Cu at (207.2, 74.6)
- renumbered BATT to J2, USB to J3, RESET to J4, RGB to J5
Connections:
- U2 pad 15: (no net) -> PROG
- U2 pad 25: (no net) -> DCCH
- U3 pad 4: (no net) -> Net-(U3-Pad4)
Routing:
- net VBUS: track 90.8 -> 493.6 mm, vias 2 -> 8
- net DATA-: track 80.3 -> 425.4 mm, vias 0 -> 2
- net DATA+: track 82.7 -> 422.9 mm, vias 0 -> 2
- net GND: track 155.7 -> 317.2 mm, vias 8 -> 9
- net Net-(D43-Pad2): track 12.7 -> 56.1 mm, vias 0 -> 1
- net Net-(F1-Pad2): track 0.00 -> 30.2 mm, vias 0 -> 3
- net Net-(U1-Pad1): track 0.00 -> 24.0 mm
- net Net-(U1-Pad3): track 0.00 -> 21.4 mm
- net Net-(D57-Pad2): track 19.8 -> 37.7 mm
- net COL13: track 295.2 -> 308.1 mm, vias 2 -> 3
- net Net-(R1-Pad2): track 0.00 -> 10.5 mm
- net Net-(R2-Pad2): track 0.00 -> 10.0 mm
- net ROW0: track 496.7 -> 499.6 mm, vias 0 -> 2
- net COL2: track 165.9 -> 168.5 mm
- net BLUE_LED: track 33.2 -> 31.3 mm
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Other:
- board size 304.8 x 119.1 mm -> 304.8 x 125.4 mm

Commit message: bit of update
Parts:
- renumbered R7 to 100K, R8 to 1K, R4 to 1K, D83 to 1N5819, R9 to 2K, R6 to 2M, R5 to 2M, R2 to 5.1K, R1 to 5.1K, F1 to 500mA, R3 to 820K, Q2 to AO3407, Q1 to AO3407, U3 to AP2112K, J2 to BATT, D82 to BLUE, D84 to RED, J4 to RESET, J5 to RGB, U4 to TP4054, U1 to USBLC6-2SC6, J3 to USB_JST, Y1 to XTAL
